File: pcb/pcb/pcb.kicad_pcb (KiCad board)
At the start: 2 copper layers, 28 parts, among them J1 Conn_01x28_Socket, J2 Conn_01x28_Socket, J3 Conn_01x03_Socket, J4 Conn_01x04_Socket, J5 MAX17048, J6 LSM6DS3TR-C, J7 SSD1306, SW1 SW_SPST, U1 TPS61022

Commit message: completed pcb
Routing:
- net +5V: track 0.00 -> 219.2 mm, vias 0 -> 10
- net GND: track 0.00 -> 182.9 mm, vias 0 -> 7
- net /PICO_SCL: track 0.00 -> 111.7 mm
- net /PICO_SDA: track 0.00 -> 103.9 mm, vias 0 -> 2
- net /GPIO0: track 0.00 -> 96.7 mm, vias 0 -> 2
- net /GPIO1: track 0.00 -> 84.1 mm, vias 0 -> 2
- net +BATT: track 0.00 -> 72.9 mm, vias 0 -> 2
- net Net-(SW1-B): track 0.00 -> 46.5 mm, vias 0 -> 2
- net /SWD: track 0.00 -> 30.6 mm, vias 0 -> 2
- net Net-(U1-FB): track 0.00 -> 30.5 mm, vias 0 -> 2
- net /GPIO8: track 0.00 -> 29.0 mm
- net /SWCLK: track 0.00 -> 28.8 mm
- net Net-(D3-DOUT): track 0.00 -> 15.7 mm
- net Net-(D1-DIN): track 0.00 -> 15.4 mm
- net Net-(U1-SW): track 0.00 -> 14.5 mm
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- added copper zone on F.Cu, net +3V3
- added copper zone on B.Cu, net GND
Other:
- board outline added: 83.5 x 129 mm
