File: pcb/pcb/pcb.kicad_pcb (KiCad board)
At the start: 2 copper layers, 83.5 x 129 mm, 28 parts, among them J1 Conn_01x28_Socket, J2 Conn_01x28_Socket, J3 Conn_01x03_Socket, J4 Conn_01x04_Socket, J5 MAX17048, J6 LSM6DS3TR-C, J7 SSD1306, SW1 SW_SPST, U1 TPS61022

Commit message: finished pcb
Parts:
- removed NT1: NetTie_2, NetTie:NetTie-2_SMD_Pad0.5mm
- added TP1: GroundTestPoint, TestPoint:TestPoint_Pad_D1.5mm, F.Cu at (69.5, 150.5)
- added TP2: BattPlusTestPoint, TestPoint:TestPoint_Pad_D1.5mm, F.Cu at (69.5, 132.8)
- added TP4: BattMinusTestPoint, TestPoint:TestPoint_Pad_D1.5mm, F.Cu at (69.5, 154.5)
- added TP5: 5VoltTestPoint, TestPoint:TestPoint_Pad_D1.5mm, F.Cu at (69.5, 137.0)
- added TP6: 3.3VoltTestPoint, TestPoint:TestPoint_Pad_D1.5mm, F.Cu at (69.5, 158.5)
- added TP7: SDATestPoint, TestPoint:TestPoint_Pad_D1.5mm, F.Cu at (69.5, 141.5)
- added TP8: SCLTestPoint, TestPoint:TestPoint_Pad_D1.5mm, F.Cu at (69.5, 162.5)
- added TP9: GPIO8TestPoint, TestPoint:TestPoint_Pad_D1.5mm, F.Cu at (69.5, 146.0)
- moved R1 2.88 mm to (90.3, 83.7)
Connections:
- C1 pad 2: GND -> -BATT
- C2 pad 2: GND -> -BATT
- C3 pad 2: GND -> -BATT
- C4 pad 2: GND -> -BATT
- C5 pad 2: GND -> -BATT
- C6 pad 2: GND -> -BATT
- C7 pad 2: GND -> -BATT
- C8 pad 2: GND -> -BATT
- D1 pad 3: GND -> -BATT
- D2 pad 3: GND -> -BATT
- D3 pad 3: GND -> -BATT
- D4 pad 3: GND -> -BATT
- J1 pad 28: GND -> -BATT
- J2 pad 28: GND -> -BATT
- J3 pad 2: GND -> -BATT
- J4 pad 3: GND -> -BATT
- J5 pad 5: GND -> -BATT
- J6 pad 7: GND -> -BATT
- J7 pad 4: GND -> -BATT
- R3 pad 2: GND -> -BATT
- R5 pad 2: GND -> -BATT
- U1 pad 1: GND -> -BATT
Routing:
- net -BATT: track 0.00 -> 190.7 mm, vias 0 -> 7
- net GND: track 185.1 -> 0.00 mm, vias 7 -> 0
- net /GPIO8: track 29.0 -> 106.8 mm, vias 0 -> 2
- net +BATT: track 72.9 -> 135.6 mm, vias 2 -> 4
- net /PICO_SCL: track 111.7 -> 156.1 mm
- net /PICO_SDA: track 103.9 -> 137.0 mm
- net +5V: track 219.2 -> 232.9 mm
- net Net-(D1-DIN): track 15.4 -> 14.2 mm
- added copper zone on B.Cu, net -BATT
- removed copper zone on B.Cu, net GND
Other:
- board text added: "Sonny and Manav"
